File: PIC16F887EV.kicad_sch (KiCad schematic)
At the start: 42 parts, among them J1 Conn_01x05_Socket, P1 USB_C_Plug_USB2.0, SW1 SW_Push, SW10 SW_Push, SW11 SW_Push, SW12 SW_Push, SW13 SW_Push, SW14 SW_Push, SW15 SW_Push, SW16 SW_Push, SW2 SW_Push, SW3 SW_Push, SW4 SW_Push, SW5 SW_Push, SW6 SW_Push, SW7 SW_Push, SW8 SW_Push, SW9 SW_Push, U1 PIC16F887-IP, U2 FT230XS

Commit message: Buzzer
Parts:
- added BZ1: Buzzer, Buzzer_Beeper:Buzzer_15x7.5RM7.6, symbol Device:Buzzer
- added C7: 100nF, Capacitor_SMD:C_1206_3216Metric_Pad1.33x1.80mm_HandSolder, symbol Device:C
- added JP1: Jumper_2_Bridged, symbol Jumper:Jumper_2_Bridged
- added R6: 330R, Resistor_SMD:R_1206_3216Metric_Pad1.30x1.75mm_HandSolder, symbol Device:R
- added U3: MMBT2222A-7-F, Downloads:SOT103P240X110-3N, symbol MMBT2222A-7-F:MMBT2222A-7-F
Connections:
- net +5V: now also BZ1.1 (-)
- net GND: now also C7.2, U3.2 (E)
- net MCLR: now also C7.1
- net RA0: now also JP1.2 (B); no longer RV1.2
- net RA3: now reaches U1.5 (C1IN+/Vref+/AN3/RA3)
- net RA3: now also R6.2
- new net: R6.1, U3.1 (B)
- new net: JP1.1 (A), RV1.2
- new net: BZ1.2 (+), U3.3 (C)
Other:
- note added: "BUZZER"
- moved on the sheet: J1, R5, RESET1

Commit message: Displays
Parts:
- added AFF1, AFF3, AFF4: LTS-6980HR, Display_7Segment:7SegmentLED_LTS6760_LTS6780, symbol Display_Character:LTS-6980HR
- added Q1, Q2, Q3: 2N3904, Package_TO_SOT_THT:TO-92_Inline, symbol Transistor_BJT:2N3904
- added R7, R8: 10K, Resistor_SMD:R_1206_3216Metric_Pad1.30x1.75mm_HandSolder, symbol Device:R
- added RD12, RD4, RD5: 4.7k, Resistor_SMD:R_1206_3216Metric_Pad1.30x1.75mm_HandSolder, symbol Device:R
- added Ra, Ra1, Ra2, Ra3, Ra4, Ra5, Ra6, Ra7: 200R, Resistor_SMD:R_1206_3216Metric_Pad1.30x1.75mm_HandSolder, symbol Device:R
- added SW17, SW18: SW_Push, Button_Switch_SMD:SW_Push_1P1T_NO_6x6mm_H9.5mm, symbol Switch:SW_Push
- JP1: footprint (none) -> Jumper:SolderJumper-2_P1.3mm_Bridged2Bar_Pad1.0x1.5mm
- RV1: footprint (none) -> Potentiometer_SMD:Potentiometer_ACP_CA6-VSMD_Vertical
Connections:
- net +5V: now also SW17.2, SW18.2
- net GND: now also Q1.1 (E), Q2.1 (E), Q3.1 (E), R7.2, R8.2
- net RD0: now also Ra.2
- net RD1: now also Ra1.2
- net RD2: now also Ra2.2
- net RD3: now also Ra3.2
- net RE2: now reaches U1.10 (RE2/AN7)
- net RE2: now also RD5.2
- net RD4: now reaches U1.27 (RD4)
- net RD4: now also Ra4.2
- net RD5: now reaches U1.28 (RD5/P1B)
- net RD5: now also Ra5.2
- net RD6: now reaches U1.29 (RD6/P1C)
- net RD6: now also Ra6.2
- net RD7: now reaches U1.30 (RD7/P1D)
- net RD7: now also Ra7.2
- net RA4: now reaches U1.6 (C1OUT/T0CKI/RA4)
- net RA4: now also R7.1, SW17.1
- net RA5: now reaches U1.7 (C2OUT/~{SS}/AN4/RA5)
- net RA5: now also R8.1, SW18.1
- net RE0: now reaches U1.8 (RE0/AN5)
- net RE0: now also RD12.2
- net RE1: now reaches U1.9 (RE1/AN6)
- net RE1: now also RD4.2
- new net: Q3.2 (B), RD5.1
- new net: AFF4.3 (C.K.), AFF4.8 (C.K.), Q3.3 (C)
- new net: Q2.2 (B), RD4.1
- new net: AFF3.3 (C.K.), AFF3.8 (C.K.), Q2.3 (C)
- new net: Q1.2 (B), RD12.1
- new net: AFF1.3 (C.K.), AFF1.8 (C.K.), Q1.3 (C)
- new net DP: AFF1.5 (DP), AFF3.5 (DP), AFF4.5 (DP), Ra7.1
- new net a: AFF1.7 (a), AFF3.7 (a), AFF4.7 (a), Ra.1
- new net b: AFF1.6 (b), AFF3.6 (b), AFF4.6 (b), Ra1.1
- new net c: AFF1.4 (c), AFF3.4 (c), AFF4.4 (c), Ra2.1
- new net d: AFF1.2 (d), AFF3.2 (d), AFF4.2 (d), Ra3.1
- new net e: AFF1.1 (e), AFF3.1 (e), AFF4.1 (e), Ra4.1
- new net f: AFF1.9 (f), AFF3.9 (f), AFF4.9 (f), Ra5.1
- new net g: AFF1.10 (g), AFF3.10 (g), AFF4.10 (g), Ra6.1
Other:
- note added: "BOTONES"
- note added: "DISPLAYS"

Commit message: Actualización
Parts:
- added AFF2: LTS-6960HR, Display_7Segment:7SegmentLED_LTS6760_LTS6780, symbol Display_Character:LTS-6960HR
- added Q4: 2N3906, Package_TO_SOT_THT:TO-92_Inline, symbol Transistor_BJT:2N3906
- added RD6: 4.7k, Resistor_SMD:R_1206_3216Metric_Pad1.30x1.75mm_HandSolder, symbol Device:R
- renumbered Ra to Ra8
Connections:
- net +5V: now also Q4.1 (E)
- net DP: now also AFF2.5 (DP)
- net ICSPCLK: now also SW11.1, SW15.1, SW3.1, SW7.1
- net ICSPDAT: now also SW12.1, SW16.1, SW4.1, SW8.1
- net RD0: no longer SW1.1, SW13.1, SW5.1, SW9.1
- net RD1: no longer SW10.1, SW14.1, SW2.1, SW6.1
- net RD2: no longer SW11.1, SW15.1, SW3.1, SW7.1
- net RD3: no longer SW12.1, SW16.1, SW4.1, SW8.1
- net RE0: now also RD6.2
- net a: now also AFF2.7 (a)
- net b: now also AFF2.6 (b)
- net c: now also AFF2.4 (c)
- net d: now also AFF2.2 (d)
- net e: now also AFF2.1 (e)
- net f: now also AFF2.9 (f)
- net g: now also AFF2.10 (g)
- net RB4: now reaches U1.37 (AN11/RB4)
- net RB4: now also SW1.1, SW13.1, SW5.1, SW9.1
- net RB5: now reaches U1.38 (~{T1G}/AN13/RB5)
- net RB5: now also SW10.1, SW14.1, SW2.1, SW6.1
- new net: Q4.2 (B), RD6.1
- new net: AFF2.3 (C.A.), AFF2.8 (C.A.), Q4.3 (C)
Other:
- note added: "DISPLAY C.A."
- moved on the sheet: AFF1, AFF3, AFF4, Q1, Q2, Q3, RD12, RD4, RD5, Ra1, Ra2, Ra3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

Commit message: Actualizacion Puente + Huellas
Agregue componentes de interfaz entre PIC (5V) y puente USB (3V3).
Cambie las huellas de transistores a SMD.
Cambie el BJT 2N2222 por un 3904
Parts:
- removed U3: MMBT2222A-7-F, Downloads:SOT103P240X110-3N, symbol MMBT2222A-7-F:MMBT2222A-7-F
- added Q5, QP1, QP2: 2N3904, Package_TO_SOT_SMD:SOT-23_Handsoldering, symbol Transistor_BJT:2N3904
- added RP10, RP8: 10K, Resistor_SMD:R_1206_3216Metric_Pad1.30x1.75mm_HandSolder, symbol Device:R
- added RP5: 2K2, Resistor_SMD:R_1206_3216Metric_Pad1.30x1.75mm_HandSolder, symbol Device:R
- added RP6: 3K3, Resistor_SMD:R_1206_3216Metric_Pad1.30x1.75mm_HandSolder, symbol Device:R
- added RP7: 4K7, Resistor_SMD:R_1206_3216Metric_Pad1.30x1.75mm_HandSolder, symbol Device:R
- added RP9: 1K, Resistor_SMD:R_1206_3216Metric_Pad1.30x1.75mm_HandSolder, symbol Device:R
- Q1, Q2, Q3, Q4: footprint Package_TO_SOT_THT:TO-92_Inline -> Package_TO_SOT_SMD:SOT-23_Handsoldering
- renumbered C1 to CP1, C2 to CP2, C3 to CP3, C4 to CP4, C5 to CP5, C6 to CP6, R2 to RP1, R1 to RP2, R3 to RP3, R4 to RP4
Connections:
- net +5V: now also RP10.1, RP8.1
- net GND: now also Q5.1 (E), QP1.1 (E), QP2.1 (E), RP6.2
- net RXpic: now also QP2.3 (C), RP10.2; no longer U2.1 (TXD)
- net TXpic: now also RP5.1; no longer U2.4 (RXD)
- net +3.3V: now reaches CP4.2, D1.2 (A), D2.2 (A), U2.10 (3V3OUT), U2.11 (~{RESET}), U2.3 (VCCIO)
- net at R6.1: now also Q5.2 (B)
- net at BZ1.2 (+): now also Q5.3 (C)
- new net: QP1.2 (B), RP7.1
- new net: RP7.2, U2.1 (TXD)
- new net: RP5.2, RP6.1, U2.4 (RXD)
- new net: QP1.3 (C), RP8.2, RP9.2
- new net: QP2.2 (B), RP9.1
Other:
- moved on the sheet: BZ1, R6

Commit message: Avance esquemático
Cristal externo + Teclado en puertos A y B con pulldown + huella potenciometro + pin de programación
Parts:
- removed AFF2: LTS-6960HR, Display_7Segment:7SegmentLED_LTS6760_LTS6780, symbol Display_Character:LTS-6960HR
- removed Q4: 2N3906, Package_TO_SOT_SMD:SOT-23_Handsoldering, symbol Transistor_BJT:2N3906
- removed RD6: 4.7k, Resistor_SMD:R_1206_3216Metric_Pad1.30x1.75mm_HandSolder, symbol Device:R
- added CP7, CP8: 47pF, Capacitor_SMD:C_1206_3216Metric_Pad1.33x1.80mm_HandSolder, symbol Device:C
- added JP2: Jumper_2_Bridged, Jumper:SolderJumper-2_P1.3mm_Bridged2Bar_Pad1.0x1.5mm, symbol Jumper:Jumper_2_Bridged
- added R1, R2, R3, R4, R9: 10K, Resistor_SMD:R_1206_3216Metric_Pad1.30x1.75mm_HandSolder, symbol Device:R
- added Y1: Crystal, Crystal:Crystal_HC18-U_Vertical, symbol Device:Crystal
- RV1: footprint Potentiometer_SMD:Potentiometer_ACP_CA6-VSMD_Vertical -> Potentiometer_SMD:Potentiometer_Vishay_TS53YL_Vertical
Connections:
- net +5V: now also JP2.1 (A)
- net GND: now also CP7.1, CP8.1, R1.2, R2.2, R3.2, R4.2, R9.2
- net ICSPCLK: no longer SW11.1, SW15.1, SW3.1, SW7.1
- net ICSPDAT: no longer SW12.1, SW16.1, SW4.1, SW8.1
- net RA0: now also SW1.1, SW13.1, SW5.1, SW9.1; no longer JP1.2 (B)
- net RA3: now also SW12.1, SW16.1, SW4.1, SW8.1; no longer R6.2
- net RA4: now also R6.2; no longer R7.1, SW17.1
- net RA5: now also JP1.2 (B); no longer R8.1, SW18.1
- net RB0: now also R1.1
- net RB1: now also R2.1
- net RB2: now also R3.1
- net RB3: now also R4.1
- net RB4: now also R7.1, SW17.1; no longer SW1.1, SW13.1, SW5.1, SW9.1
- net RB5: now also R8.1, SW18.1; no longer SW10.1, SW14.1, SW2.1, SW6.1
- net at U1.13 (RA7/OSC1/CLKIN): now also CP7.2, Y1.1
- net at U1.14 (RA6/OSC2/CLKOUT): now also CP8.2, Y1.2
- net at U1.24 (SDO/RC5): now also JP2.2 (B), R9.1
- net RA1: now reaches U1.3 (C12IN1-/AN1/RA1)
- net RA1: now also SW10.1, SW14.1, SW2.1, SW6.1
- net RA2: now reaches U1.4 (C2IN+/CVref/Vref-/AN2/RA2)
- net RA2: now also SW11.1, SW15.1, SW3.1, SW7.1
Other:
- note removed: "DISPLAY C.A."
- moved on the sheet: BZ1, C7, J1, JP1, Q5, R6, R7, R8, RESET1, RV1, SW17, SW18

Commit message: Distribución de componentes dentro del rectángulo de 10x10cm
Moví los componentes y los agrupé aproximadamente donde podrían ir dejando el PIC y el puente USB del lado inferior.
A los switchs de teclado les cambié la huella por una con modelo 3d pero del mismo footprint
Parts:
- RESET1: footprint Button_Switch_SMD:SW_Push_1P1T_NO_6x6mm_H9.5mm -> Button_Switch_SMD:SW_SPST_TL3342
- SW1, SW10, SW11, SW12, SW13, SW14, SW15, SW16, SW17, SW18, SW2, SW3, SW4, SW5, SW6, SW7, SW8, SW9: footprint Button_Switch_SMD:SW_Push_1P1T_NO_6x6mm_H9.5mm -> Button_Switch_SMD:SW_SPST_PTS645
Changed lines of the file:
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@@
       (effects (font (size 1.27 1.27)))
     )
-    (property "Footprint" "Button_Switch_SMD:SW_Push_1P1T_NO_6x6mm_H9.5mm" (at 355.6 69.85 0)
+    (property "Footprint" "Button_Switch_SMD:SW_SPST_PTS645" (at 355.6 69.85 0)
       (effects (font (size 1.27 1.27)) hide)
     )
@@
       (effects (font (size 1.27 1.27)))
     )
-    (property "Footprint" "Button_Switch_SMD:SW_Push_1P1T_NO_6x6mm_H9.5mm" (at 378.46 69.85 0)
+    (property "Footprint" "Button_Switch_SMD:SW_SPST_PTS645" (at 378.46 69.85 0)
       (effects (font (size 1.27 1.27)) hide)
     )
@@
       (effects (font (size 1.27 1.27)))
     )
-    (property "Footprint" "Button_Switch_SMD:SW_Push_1P1T_NO_6x6mm_H9.5mm" (at 378.46 53.34 0)
+    (property "Footprint" "Button_Switch_SMD:SW_SPST_PTS645" (at 378.46 53.34 0)
       (effects (font (size 1.27 1.27)) hide)
     )
@@
       (effects (font (size 1.27 1.27)))
     )
-    (property "Footprint" "Button_Switch_SMD:SW_Push_1P1T_NO_6x6mm_H9.5mm" (at 355.6 53.34 0)
+    (property "Footprint" "Button_Switch_SMD:SW_SPST_PTS645" (at 355.6 53.34 0)
       (effects (font (size 1.27 1.27)) hide)
     )
@@
       (effects (font (size 1.27 1.27)))
     )
-    (property "Footprint" "Button_Switch_SMD:SW_Push_1P1T_NO_6x6mm_H9.5mm" (at 312.42 53.34 0)
+    (property "Footprint" "Button_Switch_SMD:SW_SPST_PTS645" (at 312.42 53.34 0)
       (effects (font (size 1.27 1.27)) hide)
     )
@@
       (effects (font (size 1.27 1.27)))
     )
-    (property "Footprint" "Button_Switch_SMD:SW_Push_1P1T_NO_6x6mm_H9.5mm" (at 378.46 36.83 0)
+    (property "Footprint" "Button_Switch_SMD:SW_SPST_PTS645" (at 378.46 36.83 0)
       (effects (font (size 1.27 1.27)) hide)
     )
@@
       (effects (font (size 1.27 1.27)))
     )
-    (property "Footprint" "Button_Switch_SMD:SW_Push_1P1T_NO_6x6mm_H9.5mm" (at 312.42 69.85 0)
+    (property "Footprint" "Button_Switch_SMD:SW_SPST_PTS645" (at 312.42 69.85 0)
       (effects (font (size 1.27 1.27)) hide)
     )
@@
       (effects (font (size 1.27 1.27)) (justify right))
     )
-    (property "Footprint" "Button_Switch_SMD:SW_Push_1P1T_NO_6x6mm_H9.5mm" (at 34.29 78.74 0)
+    (property "Footprint" "Button_Switch_SMD:SW_SPST_TL3342" (at 34.29 78.74 0)
       (effects (font (size 1.27 1.27)) hide)
     )
@@
       (effects (font (size 1.27 1.27)))
     )
-    (property "Footprint" "Button_Switch_SMD:SW_Push_1P1T_NO_6x6mm_H9.5mm" (at 334.01 69.85 0)
+    (property "Footprint" "Button_Switch_SMD:SW_SPST_PTS645" (at 334.01 69.85 0)
       (effects (font (size 1.27 1.27)) hide)
     )
@@
       (effects (font (size 1.27 1.27)))
     )
-    (property "Footprint" "Button_Switch_SMD:SW_Push_1P1T_NO_6x6mm_H9.5mm" (at 355.6 36.83 0)
+    (property "Footprint" "Button_Switch_SMD:SW_SPST_PTS645" (at 355.6 36.83 0)
       (effects (font (size 1.27 1.27)) hide)
     )
@@
       (effects (font (size 1.27 1.27)))
     )
-    (property "Footprint" "Button_Switch_SMD:SW_Push_1P1T_NO_6x6mm_H9.5mm" (at 378.46 85.09 0)
+    (property "Footprint" "Button_Switch_SMD:SW_SPST_PTS645" (at 378.46 85.09 0)
       (effects (font (size 1.27 1.27)) hide)
     )
@@
       (effects (font (size 1.27 1.27)))
     )
-    (property "Footprint" "Button_Switch_SMD:SW_Push_1P1T_NO_6x6mm_H9.5mm" (at 334.01 36.83 0)
+    (property "Footprint" "Button_Switch_SMD:SW_SPST_PTS645" (at 334.01 36.83 0)
       (effects (font (size 1.27 1.27)) hide)
     )
@@
       (effects (font (size 1.27 1.27)))
     )
-    (property "Footprint" "Button_Switch_SMD:SW_Push_1P1T_NO_6x6mm_H9.5mm" (at 312.42 36.83 0)
+    (property "Footprint" "Button_Switch_SMD:SW_SPST_PTS645" (at 312.42 36.83 0)
       (effects (font (size 1.27 1.27)) hide)
     )
@@
       (effects (font (size 1.27 1.27)))
     )
-    (property "Footprint" "Button_Switch_SMD:SW_Push_1P1T_NO_6x6mm_H9.5mm" (at 334.01 85.09 0)
+    (property "Footprint" "Button_Switch_SMD:SW_SPST_PTS645" (at 334.01 85.09 0)
       (effects (font (size 1.27 1.27)) hide)
     )
@@
       (effects (font (size 1.27 1.27)))
     )
-    (property "Footprint" "Button_Switch_SMD:SW_Push_1P1T_NO_6x6mm_H9.5mm" (at 334.01 53.34 0)
+    (property "Footprint" "Button_Switch_SMD:SW_SPST_PTS645" (at 334.01 53.34 0)
       (effects (font (size 1.27 1.27)) hide)
     )
@@
       (effects (font (size 1.27 1.27)))
     )
-    (property "Footprint" "Button_Switch_SMD:SW_Push_1P1T_NO_6x6mm_H9.5mm" (at 273.05 31.115 0)
+    (property "Footprint" "Button_Switch_SMD:SW_SPST_PTS645" (at 273.05 31.115 0)
       (effects (font (size 1.27 1.27)) hide)
     )
@@
       (effects (font (size 1.27 1.27)))
     )
-    (property "Footprint" "Button_Switch_SMD:SW_Push_1P1T_NO_6x6mm_H9.5mm" (at 312.42 85.09 0)
+    (property "Footprint" "Button_Switch_SMD:SW_SPST_PTS645" (at 312.42 85.09 0)
       (effects (font (size 1.27 1.27)) hide)
     )
@@
       (effects (font (size 1.27 1.27)))
     )
-    (property "Footprint" "Button_Switch_SMD:SW_Push_1P1T_NO_6x6mm_H9.5mm" (at 240.03 31.115 0)
+    (property "Footprint" "Button_Switch_SMD:SW_SPST_PTS645" (at 240.03 31.115 0)
       (effects (font (size 1.27 1.27)) hide)
     )
@@
       (effects (font (size 1.27 1.27)))
     )
-    (property "Footprint" "Button_Switch_SMD:SW_Push_1P1T_NO_6x6mm_H9.5mm" (at 355.6 85.09 0)
-      (effects (font (size 1.27 1.27)) hide)
-    )
+    (property "Footprint" "Button_Switch_SMD:SW_SPST_PTS645" (at 355.6 85.09 0)
+      (effects (font (size 1.27 1.27)) hide)
+    )
